File: Kicad/QPL9065.sch (KiCad schematic (older format))
At the start: 24 parts, among them J1 Conn_Coaxial, J2 Conn_Coaxial, J3 Conn_Coaxial_Power, U1 QPL9065

Commit message: Shield line, new footprint, cleanup
Parts:
- U1: footprint Package_DFN_QFN:QFN-16-1EP_3x3mm_P0.5mm_EP2.7x2.7mm_ThermalVias -> Package_DFN_QFN:UQFN-16-1EP_3x3mm_P0.5mm_QPL9065
Changed lines of the file:
@@
 F 0 "U1" H 5500 3750 50  0000 L CNN
 F 1 "QPL9065" H 5400 3650 50  0000 L CNN
-F 2 "Package_DFN_QFN:QFN-16-1EP_3x3mm_P0.5mm_EP2.7x2.7mm_ThermalVias" H 5600 3800 50  0001 C CNN
+F 2 "Package_DFN_QFN:UQFN-16-1EP_3x3mm_P0.5mm_QPL9065" H 5600 3800 50  0001 C CNN
 F 3 "" H 5600 3800 50  0001 C CNN
 	1    5600 3750

Commit message: Case, Impedence matchine LNA
Parts:
- J1, J2: footprint Connector_Coaxial:SMA_Amphenol_132289_EdgeMount-RF -> Connector_Coaxial:‎142-1701-626‎
- J3: symbol Connector:Conn_Coaxial_Power -> Connector:132147-48
Changed lines of the file:
@@
 F 0 "J1" H 3200 3800 50  0000 C CNN
 F 1 "Conn_Coaxial" H 3400 3700 50  0001 C CNN
-F 2 "Connector_Coaxial:SMA_Amphenol_132289_EdgeMount-RF" H 3050 3750 50  0001 C CNN
+F 2 "Connector_Coaxial:‎142-1701-626‎" H 3050 3750 50  0001 C CNN
 F 3 " ~" H 3050 3750 50  0001 C CNN
 	1    3050 3750
@@
 F 0 "J2" H 8050 3800 50  0000 L CNN
 F 1 "Conn_Coaxial" H 8050 3700 50  0001 L CNN
-F 2 "Connector_Coaxial:SMA_Amphenol_132289_EdgeMount-RF" H 7950 3750 50  0001 C CNN
+F 2 "Connector_Coaxial:‎142-1701-626‎" H 7950 3750 50  0001 C CNN
 F 3 " ~" H 7950 3750 50  0001 C CNN
 	1    7950 3750
@@
 	4150 3150 4650 3150
 $Comp
-L Connector:Conn_Coaxial_Power J3
+L Connector:132147-48 J3
 U 1 1 5FDD017F
 P 5600 2300

Commit message: Update 50ohm FR4 Er 4.03
Parts:
- J3: footprint Connector_Coaxial:SMA_Amphenol_132289_EdgeMount-RF -> Connector_Coaxial:132147-48
Changed lines of the file:
@@
 F 0 "J3" H 5688 2250 50  0000 L CNN
 F 1 "Conn_Coaxial_Power" H 5688 2205 50  0001 L CNN
-F 2 "Connector_Coaxial:SMA_Amphenol_132289_EdgeMount-RF" H 5600 2250 50  0001 C CNN
+F 2 "Connector_Coaxial:132147-48" H 5600 2250 50  0001 C CNN
 F 3 "~" H 5600 2250 50  0001 C CNN
 	1    5600 2300
